File: Skeuomorphic_candle_digital/Skeuomorphic_candle_digital.kicad_sch (KiCad schematic)
At the start: 19 parts, among them J2 Conn_01x02_Pin, Q1 SI2302, U2 CH32V003JxMx

Commit message: added readme per pcb variant. fixed some component values
Parts:
- R1: value 100k -> 47k
Changed lines of the file:
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@@
 			)
 		)
-		(property "Value" "100k"
+		(property "Value" "47k"
 			(at 44.45 68.5799 0)
 			(show_name no)
